File: cad/pcb/mainboard/power.kicad_sch (KiCad schematic)
At the start: 0 parts

Commit message: more schematic work
Parts:
- added C43: 3.3u, symbol Device:C
- added C44: 100n, symbol Device:C
- added C45: 56p, symbol Device:C
- added C46: 47u, symbol Device:C
- added L1: L, symbol Device:L
- added Q1, Q2: IRLZ44N, Package_TO_SOT_THT:TO-220-3_Vertical, symbol Transistor_FET:IRLZ44N
- added R27: 100k, symbol Device:R
- added R28: 22.1k, symbol Device:R
- added U8: TPS54202DDC, Package_TO_SOT_SMD:SOT-23-6, symbol Regulator_Switching:TPS54202DDC
Connections:
- new net: C45.1, R27.2, R28.1, U8.4 (FB)
- new net: C44.1, U8.6 (BOOT)
- new net: C44.2, L1.1, U8.2 (SW)
- new net +3.3V: C45.2, C46.2, L1.2, R27.1
- new net +BED: C43.1, U8.3 (VIN)
- new net -BED: Q1.2 (D)
- new net -NOZ: Q2.2 (D)
- new net GND: C43.2, C46.1, Q1.3 (S), Q2.3 (S), R28.2, U8.1 (GND)
- new net PWM_BED: Q1.1 (G)
- new net PWM_NOZ: Q2.1 (G)

Commit message: cad and kicad progress
Parts:
- added TP17, TP18: TestPoint, symbol Connector:TestPoint
- L1: value L -> 3.9uH 70mOhm
Connections:
- net +3.3V: now also TP18.1
- net +BED: now also TP17.1
- no-connect marks 0 -> 1
Changed lines of the file:
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@@
 	(paper "A4")
+	(junction
+		(at 35.56 36.83)
+		(diameter 0)
+		(color 0 0 0 0)
+	)
 	(junction
 		(at 118.11 90.17)
@@
 		(color 0 0 0 0)
 	)
+	(junction
+		(at 35.56 25.4)
+		(diameter 0)
+		(color 0 0 0 0)
+	)
+	(no_connect
+		(at 52.07 80.01)
+	)
 	(wire
 		(pts
@@
 	(wire
 		(pts
-			(xy 34.29 36.83) (xy 40.64 36.83)
+			(xy 31.75 36.83) (xy 35.56 36.83)
 		)
 		(stroke
@@
 	(wire
 		(pts
+			(xy 35.56 36.83) (xy 35.56 40.64)
+		)
+		(stroke
+			(width 0)
+			(type default)
+		)
+	)
+	(wire
+		(pts
 			(xy 256.54 58.42) (xy 256.54 57.15)
 		)
@@
 	(wire
 		(pts
-			(xy 38.1 29.21) (xy 34.29 29.21)
+			(xy 38.1 25.4) (xy 35.56 25.4)
 		)
 		(stroke
@@
 	(wire
 		(pts
+			(xy 35.56 36.83) (xy 38.1 36.83)
+		)
+		(stroke
+			(width 0)
+			(type default)
+		)
+	)
+	(wire
+		(pts
 			(xy 113.03 74.93) (xy 123.19 74.93)
 		)
@@
 	(wire
 		(pts
+			(xy 35.56 25.4) (xy 34.29 25.4)
+		)
+		(stroke
+			(width 0)
+			(type default)
+		)
+	)
+	(wire
+		(pts
 			(xy 95.25 74.93) (xy 100.33 74.93)
 		)
@@
 	(wire
 		(pts
+			(xy 35.56 17.78) (xy 38.1 17.78)
+		)
+		(stroke
+			(width 0)
+			(type default)
+		)
+	)
+	(wire
+		(pts
 			(xy 118.11 90.17) (xy 123.19 90.17)
 		)
@@
 	(wire
 		(pts
+			(xy 35.56 25.4) (xy 35.56 17.78)
+		)
+		(stroke
+			(width 0)
+			(type default)
+		)
+	)
+	(wire
+		(pts
 			(xy 100.33 74.93) (xy 113.03 74.93)
 		)
@@
 	)
 	(label "VBUS"
-		(at 38.1 29.21 0)
+		(at 38.1 25.4 0)
 		(effects
 			(font
@@
 	(hierarchical_label "VBUS"
 		(shape input)
-		(at 34.29 29.21 180)
+		(at 34.29 25.4 180)
 		(effects
 			(font
@@
 	(hierarchical_label "3V3"
 		(shape output)
-		(at 40.64 36.83 0)
+		(at 38.1 36.83 0)
 		(effects
 			(font
@@
 	(symbol
 		(lib_id "power:+3.3V")
-		(at 34.29 36.83 0)
+		(at 31.75 36.83 0)
 		(unit 1)
 		(exclude_from_sim no)
@@
 		(fields_autoplaced yes)
 		(property "Reference" "#PWR080"
-			(at 34.29 40.64 0)
+			(at 31.75 40.64 0)
 			(effects
 				(font
@@
 		)
 		(property "Value" "+3.3V"
-			(at 34.29 31.75 0)
+			(at 31.75 31.75 0)
 			(effects
 				(font
@@
 		)
 		(property "Footprint" ""
-			(at 34.29 36.83 0)
+			(at 31.75 36.83 0)
 			(effects
 				(font
@@
 		)
 		(property "Datasheet" ""
-			(at 34.29 36.83 0)
+			(at 31.75 36.83 0)
 			(effects
 				(font
@@
 		)
 		(property "Description" "Power symbol creates a global label with name \"+3.3V\""
-			(at 34.29 36.83 0)
+			(at 31.75 36.83 0)
 			(effects
 				(font
@@
 	)
 	(symbol
+		(lib_id "Connector:TestPoint")
+		(at 35.56 40.64 270)
+		(unit 1)
+		(exclude_from_sim no)
+		(in_bom yes)
+		(on_board yes)
+		(dnp no)
+		(property "Reference" "TP18"
+			(at 38.862 43.434 90)
+			(effects
+				(font
+					(size 1.27 1.27)
+				)
+			)
+		)
+		(property "Value" "TestPoint"
+			(at 38.862 43.18 90)
+			(effects
+				(font
+					(size 1.27 1.27)
+				)
+				(hide yes)
+			)
+		)
+		(property "Footprint" ""
+			(at 35.56 45.72 0)
+			(effects
+				(font
+					(size 1.27 1.27)
+				)
+				(hide yes)
+			)
+		)
+		(property "Datasheet" "~"
+			(at 35.56 45.72 0)
+			(effects
+				(font
+					(size 1.27 1.27)
+				)
+				(hide yes)
+			)
+		)
+		(property "Description" "test point"
+			(at 35.56 40.64 0)
+			(effects
+				(font
+					(size 1.27 1.27)
+				)
+				(hide yes)
+			)
+		)
+		(pin "1"
+		)
+		(instances
+			(project "mainboard"
+				(path "/2af8450f-8363-4132-8171-0f0f10c5c429/f2927a02-2577-43d8-8597-6ea8a6a0445d"
+					(reference "TP18")
+					(unit 1)
+				)
+			)
+		)
+	)
+	(symbol
 		(lib_id "power:GND")
 		(at 35.56 83.82 0)
@@
 			)
 		)
-		(property "Value" "L"
+		(property "Value" "3.9uH 70mOhm"
 			(at 91.44 72.39 90)
 			(effects
@@
 					(unit 1)
 				)
+			)
+		)
+	)
+	(symbol
+		(lib_id "Connector:TestPoint")
+		(at 38.1 17.78 270)
+		(unit 1)
+		(exclude_from_sim no)
+		(in_bom yes)
+		(on_board yes)
+		(dnp no)
+		(property "Reference" "TP17"
+			(at 41.402 20.574 90)
+			(effects
+				(font
+					(size 1.27 1.27)
+				)
+			)
+		)
+		(property "Value" "TestPoint"
+			(at 41.402 20.32 90)
+			(effects
+				(font
+					(size 1.27 1.27)
+				)
+				(hide yes)
+			)
+		)
+		(property "Footprint" ""
+			(at 38.1 22.86 0)
+			(effects
+				(font
+					(size 1.27 1.27)
+				)
+				(hide yes)
+			)
+		)
+		(property "Datasheet" "~"
+			(at 38.1 22.86 0)
+			(effects
+				(font
+					(size 1.27 1.27)
+				)
+				(hide yes)
+			)
+		)
+		(property "Description" "test point"
+			(at 38.1 17.78 0)
+			(effects
+				(font
+					(size 1.27 1.27)
+				)
+				(hide yes)
+			)
+		)
+		(pin "1"
+		)
+		(instances
+			(project "mainboard"
+				(path "/2af8450f-8363-4132-8171-0f0f10c5c429/f2927a02-2577-43d8-8597-6ea8a6a0445d"
+					(reference "TP17")
+					(unit 1)
+				)
