File: cad/pcb/mainboard/untitled.kicad_sch (KiCad schematic)
At the start: 6 parts

Commit message: cad and kicad progress
Changed lines of the file:
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@@
 	(wire
 		(pts
-			(xy 215.9 46.99) (xy 223.52 46.99)
+			(xy 205.74 91.44) (xy 213.36 91.44)
 		)
 		(stroke
@@
 	(wire
 		(pts
-			(xy 217.17 27.94) (xy 224.79 27.94)
+			(xy 207.01 72.39) (xy 214.63 72.39)
 		)
 		(stroke
@@
 	(wire
 		(pts
-			(xy 215.9 20.32) (xy 224.79 20.32)
+			(xy 205.74 64.77) (xy 214.63 64.77)
 		)
 		(stroke
@@
 	(wire
 		(pts
-			(xy 215.9 43.18) (xy 223.52 43.18)
-		)
-		(stroke
-			(width 0)
-			(type default)
-		)
-	)
-	(wire
-		(pts
-			(xy 217.17 34.29) (xy 224.79 34.29)
+			(xy 205.74 87.63) (xy 213.36 87.63)
+		)
+		(stroke
+			(width 0)
+			(type default)
+		)
+	)
+	(wire
+		(pts
+			(xy 207.01 78.74) (xy 214.63 78.74)
 		)
 		(stroke
@@
 	)
 	(label "~{EN}"
-		(at 217.17 34.29 0)
+		(at 207.01 78.74 0)
 		(effects
 			(font
@@
 	)
 	(label "UART1"
-		(at 215.9 43.18 0)
+		(at 205.74 87.63 0)
 		(effects
 			(font
@@
 	)
 	(label "UART2"
-		(at 215.9 46.99 0)
+		(at 205.74 91.44 0)
 		(effects
 			(font
@@
 	)
 	(label "VBUS"
-		(at 215.9 20.32 0)
+		(at 205.74 64.77 0)
 		(effects
 			(font
@@
 	(hierarchical_label "~{EN}"
 		(shape input)
-		(at 224.79 34.29 0)
+		(at 214.63 78.74 0)
 		(effects
 			(font
@@
 	(hierarchical_label "UART2"
 		(shape bidirectional)
-		(at 223.52 46.99 0)
+		(at 213.36 91.44 0)
 		(effects
 			(font
@@
 	(hierarchical_label "3V3"
 		(shape input)
-		(at 224.79 27.94 0)
+		(at 214.63 72.39 0)
 		(effects
 			(font
@@
 	(hierarchical_label "UART1"
 		(shape bidirectional)
-		(at 223.52 43.18 0)
+		(at 213.36 87.63 0)
 		(effects
 			(font
@@
 	(hierarchical_label "VBUS"
 		(shape input)
-		(at 224.79 20.32 0)
+		(at 214.63 64.77 0)
 		(effects
 			(font
@@
 	(symbol
 		(lib_id "power:+3.3V")
-		(at 217.17 27.94 0)
+		(at 207.01 72.39 0)
 		(unit 1)
 		(exclude_from_sim no)
@@
 		(fields_autoplaced yes)
 		(property "Reference" "#PWR017"
-			(at 217.17 31.75 0)
+			(at 207.01 76.2 0)
 			(effects
 				(font
@@
 		)
 		(property "Value" "+3.3V"
-			(at 217.17 22.86 0)
+			(at 207.01 67.31 0)
 			(effects
 				(font
@@
 		)
 		(property "Footprint" ""
-			(at 217.17 27.94 0)
+			(at 207.01 72.39 0)
 			(effects
 				(font
@@
 		)
 		(property "Datasheet" ""
-			(at 217.17 27.94 0)
+			(at 207.01 72.39 0)
 			(effects
 				(font
@@
 		)
 		(property "Description" "Power symbol creates a global label with name \"+3.3V\""
-			(at 217.17 27.94 0)
-			(effects
-				(font
+			(at 207.01 72.39 0)
+			(effects
+				(font
