File: cad/pcb/mainboard/mainboard.kicad_sch (KiCad schematic)
At the start: 0 parts

Commit message: more schematic work
Parts:
- added BED, NOZ, VBUS: Conn_01x02_Socket, symbol Connector:Conn_01x02_Socket
- added J3: USB_C_Receptacle_USB2.0_16P, Connector_USB:USB_C_Receptacle_GCT_USB4105-xx-A_16P_TopMnt_Horizontal, symbol Connector:USB_C_Receptacle_USB2.0_16P
Connections:
- new net: J3.A1 (GND), J3.A12 (GND), J3.B1 (GND), J3.B12 (GND)
- new net: J3.A4 (VBUS), J3.A9 (VBUS), J3.B4 (VBUS), J3.B9 (VBUS)
- new net GND: VBUS.1 (Pin_1)
- new net VBUS: VBUS.2 (Pin_2)
- new net power/+BED: BED.2 (Pin_2)
- new net power/+NOZ: NOZ.2 (Pin_2)
- new net power/-BED: BED.1 (Pin_1)
- new net power/-NOZ: NOZ.1 (Pin_1)
- new net stm32/D+: J3.A6 (D+), J3.B6 (D+)
- new net stm32/D-: J3.A7 (D-), J3.B7 (D-)
Other:
- sheet power ports: added +BED, +NOZ, -BED, -NOZ, 3V3, PWM_BED, PWM_NOZ, VBUS; removed none
- sheet stm32 ports: added D+, D-, VMCU; removed none

Commit message: cad and kicad progress
Parts:
- added C54, C55: 100n, symbol Device:C
- added HMI: Conn_01x05_Pin, symbol Connector:Conn_01x05_Pin
- added R31, R32: 10k, symbol Device:R
- added R33: 1M, symbol Device:R
- added TBED, TNOZ: Conn_01x02_Pin, symbol Connector:Conn_01x02_Pin
- added TP13, TP14, TP15, TP16: TestPoint, symbol Connector:TestPoint
Connections:
- net +3.3V: now also HMI.2 (Pin_2), R31.2, R32.2
- net GND: now also J3.A1 (GND), J3.A12 (GND), J3.B1 (GND), J3.B12 (GND), C54.2, C55.2, HMI.1 (Pin_1), R33.2, TBED.1 (Pin_1), TNOZ.1 (Pin_1)
- net power/PWM_BED: now also TP16.1
- net power/PWM_NOZ: now also TP15.1
- net at J3.S1 (SHIELD): now also R33.1
- new net TBED: C55.1, R32.1, TBED.2 (Pin_2), TP13.1
- new net TNOZ: C54.1, R31.1, TNOZ.2 (Pin_2), TP14.1
- new net stm32/HMI_RST: HMI.5 (Pin_5)
- new net stm32/HMI_RX: HMI.4 (Pin_4)
- new net stm32/HMI_TX: HMI.3 (Pin_3)
Other:
- sheet stm32 ports: added HMI_RST, HMI_RX, HMI_TX, PWM_BED, PWM_NOZ, TBED, TNOZ; removed none
- moved on the sheet: J3

Commit message: cad work today
Parts:
- added R34, R35: 5.1k, symbol Device:R
Connections:
- net GND: now also R34.2, R35.1
- net at J3.A5 (CC1): now also R35.2
- net at J3.B5 (CC2): now also R34.1
- no-connect marks 0 -> 2
