File: cad/pcb/mainboard/stm32.kicad_sch (KiCad schematic)
At the start: 3 parts, among them U7 STM32G431CBTx

Commit message: more schematic work
Parts:
- added C47, C48: C, symbol Device:C
- added Y1: Crystal, symbol Device:Crystal
Changed lines of the file:
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@@
+		)
+	)
+	(hierarchical_label "VMCU"
+		(shape input)
+		(at 81.28 59.69 0)
+		(effects
+			(font
+				(size 1.27 1.27)
+			)
+			(justify left)
+		)
+	)
+	(hierarchical_label "D+"
+		(shape bidirectional)
+		(at 68.58 116.84 180)
+		(effects
+			(font
+				(size 1.27 1.27)
+			)
+			(justify right)
+		)
+	)
+	(hierarchical_label "D-"
+		(shape bidirectional)
+		(at 68.58 113.03 180)
+		(effects
+			(font
+				(size 1.27 1.27)
+			)
+			(justify right)
 		)
 	)
@@
 	)
 	(symbol
+		(lib_id "Device:Crystal")
+		(at 111.76 100.33 0)
+		(unit 1)
+		(exclude_from_sim no)
+		(in_bom yes)
+		(on_board yes)
+		(dnp no)
+		(fields_autoplaced yes)
+		(property "Reference" "Y1"
+			(at 111.76 92.71 0)
+			(effects
+				(font
+					(size 1.27 1.27)
+				)
+			)
+		)
+		(property "Value" "Crystal"
+			(at 111.76 95.25 0)
+			(effects
+				(font
+					(size 1.27 1.27)
+				)
+			)
+		)
+		(property "Footprint" ""
+			(at 111.76 100.33 0)
+			(effects
+				(font
+					(size 1.27 1.27)
+				)
+				(hide yes)
+			)
+		)
+		(property "Datasheet" "~"
+			(at 111.76 100.33 0)
+			(effects
+				(font
+					(size 1.27 1.27)
+				)
+				(hide yes)
+			)
+		)
+		(property "Description" "Two pin crystal"
+			(at 111.76 100.33 0)
+			(effects
+				(font
+					(size 1.27 1.27)
+				)
+				(hide yes)
+			)
+		)
+		(pin "2"
+		)
+		(pin "1"
+		)
+		(instances
+			(project ""
+				(path "/2af8450f-8363-4132-8171-0f0f10c5c429/5c64e139-f759-4e48-a9a5-8c1e03f8a77c"
+					(reference "Y1")
+					(unit 1)
+				)
+			)
+		)
+	)
+	(symbol
+		(lib_id "Device:C")
+		(at 104.14 109.22 0)
+		(unit 1)
+		(exclude_from_sim no)
+		(in_bom yes)
+		(on_board yes)
+		(dnp no)
+		(fields_autoplaced yes)
+		(property "Reference" "C47"
+			(at 107.95 107.9499 0)
+			(effects
+				(font
+					(size 1.27 1.27)
+				)
+				(justify left)
+			)
+		)
+		(property "Value" "C"
+			(at 107.95 110.4899 0)
+			(effects
+				(font
+					(size 1.27 1.27)
+				)
+				(justify left)
+			)
+		)
+		(property "Footprint" ""
+			(at 105.1052 113.03 0)
+			(effects
+				(font
+					(size 1.27 1.27)
+				)
+				(hide yes)
+			)
+		)
+		(property "Datasheet" "~"
+			(at 104.14 109.22 0)
+			(effects
+				(font
+					(size 1.27 1.27)
+				)
+				(hide yes)
+			)
+		)
+		(property "Description" "Unpolarized capacitor"
+			(at 104.14 109.22 0)
+			(effects
+				(font
+					(size 1.27 1.27)
+				)
+				(hide yes)
+			)
+		)
+		(pin "2"
+		)
+		(pin "1"
+		)
+		(instances
+			(project ""
+				(path "/2af8450f-8363-4132-8171-0f0f10c5c429/5c64e139-f759-4e48-a9a5-8c1e03f8a77c"
+					(reference "C47")
+					(unit 1)
+				)
+			)
+		)
+	)
+	(symbol
 		(lib_id "Device:R")
 		(at 50.8 43.18 90)
@@
 					(unit 1)
 				)
+			)
+		)
+	)
+	(symbol
+		(lib_id "Device:C")
+		(at 116.84 109.22 0)
+		(unit 1)
+		(exclude_from_sim no)
+		(in_bom yes)
+		(on_board yes)
+		(dnp no)
+		(fields_autoplaced yes)
+		(property "Reference" "C48"
+			(at 120.65 107.9499 0)
+			(effects
+				(font
+					(size 1.27 1.27)
+				)
+				(justify left)
+			)
+		)
+		(property "Value" "C"
+			(at 120.65 110.4899 0)
+			(effects
+				(font
+					(size 1.27 1.27)
+				)
+				(justify left)
+			)
+		)
+		(property "Footprint" ""
+			(at 117.8052 113.03 0)
+			(effects
+				(font
+					(size 1.27 1.27)
+				)
+				(hide yes)
+			)
+		)
+		(property "Datasheet" "~"
+			(at 116.84 109.22 0)
+			(effects
+				(font
+					(size 1.27 1.27)
+				)
+				(hide yes)
+			)
+		)
+		(property "Description" "Unpolarized capacitor"
+			(at 116.84 109.22 0)
+			(effects
+				(font
+					(size 1.27 1.27)
+				)
+				(hide yes)
+			)
+		)
+		(pin "1"
+		)
+		(pin "2"
+		)
+		(instances
+			(project ""
+				(path "/2af8450f-8363-4132-8171-0f0f10c5c429/5c64e139-f759-4e48-a9a5-8c1e03f8a77c"
+					(reference "C48")
+					(unit 1)
+				)

Commit message: cad and kicad progress
Parts:
- removed Y1: Crystal, symbol Device:Crystal
- added C49: 1u, symbol Device:C
- added C50: 10n, symbol Device:C
- added C51, C52, C53: 100n, symbol Device:C
- added FB1: FerriteBead, symbol Device:FerriteBead
- added R29, R30: 22, symbol Device:R
- added Y2: Crystal_GND24, symbol Device:Crystal_GND24
- C47, C48: value C -> 22p
Connections:
- net D+: now also R30.1
- net D-: now also R29.1
- net GND: now reaches C47.1
- net GND: now also C48.1, U7.19 (VSSA), U7.23 (VSS), U7.35 (VSS), U7.47 (VSS), C49.2, C50.2, C51.2, C52.2, C53.2, Y2.2, Y2.4
- net at C47.2: now also U7.5 (PF0), Y2.3
- net at C48.2: now also U7.6 (PF1), Y2.1
- net +3.3V: now reaches U7.1 (VBAT)
- net +3.3V: now also U7.24 (VDD), U7.36 (VDD), U7.48 (VDD), C51.1, C52.1, C53.1, FB1.1
- net +3.3VA: now reaches U7.20 (VREF+)
- net +3.3VA: now also U7.21 (VDDA), C49.1, C50.1, FB1.2
Other:
- note added: "MCU VDD caps"
- moved on the sheet: C47, C48

Commit message: cad work today
Parts:
- removed Y2: Crystal_GND24, symbol Device:Crystal_GND24
- added Y1: X322516MLB4SI, Crystal:Crystal_SMD_3225-4Pin_3.2x2.5mm, symbol Device:Crystal_GND24
- C47, C48: value 22p -> 12p
Connections:
- net GND: now also Y1.2, Y1.4
- net at R29.2: now also U7.33 (PA11)
- net at R30.2: now also U7.34 (PA12)
- net at C47.2, U7.5 (PF0): now also Y1.3
- net at C48.2, U7.6 (PF1): now also Y1.1
Other:
- moved on the sheet: R29, R30
